Commit message: added mpu6050 and use imu as odometry sensor

File: bumperbot_ws/src/bumperbot_bringup/urdf/bumperbot_gazebo.xacro (robot description, xacro)
@@ -3,7 +3,6 @@
 <gazebo>
     <plugin name="gazebo_ros2_control" filename="libgazebo_ros2_control.so">
-        <!-- <parameters>$(find bumperbot_controller)/config/my_control.yaml</parameters> -->
-        <parameters>$(find bumperbot_bringup)/config/bumperbot_bringup.yaml</parameters>
-        <!-- <parameters>$(find techmon_controller)/config/gazebo_ros2_ctl_use_sim.yaml</parameters> -->
+        <parameters>$(find bumperbot_bringup)/config/bumperbot_controllers.yaml</parameters>
+        <!-- <parameters>$(find bumperbot_bringup)/config/bumperbot_bringup.yaml</parameters> -->
     </plugin>
 </gazebo>

File: bumperbot_ws/src/bumperbot_bringup/urdf/rover.xacro (robot description, xacro)
@@ -198,4 +198,30 @@
     <gazebo reference="ldlidar_link">
         <material>Gazebo/Blue</material>
+    </gazebo>
+    <!-- IMU JOINT -->
+    <joint name="imu_joint" type="fixed">
+        <origin xyz="0.0 0.0 0.015 " rpy="0.0 0.0 0.0"/>
+        <parent link="ldlidar_link"/>
+        <child link="imu_link"/>
+    </joint>
+    <!-- IMU LINK -->
+    <link name="imu_link">
+    <visual>
+        <geometry>
+            <cylinder radius="0.01" length="0.01"/>
+        </geometry>
+        <material name="white"/>
+    </visual>
+    <collision>
+        <geometry>
+            <cylinder radius="0.01" length="0.01"/>
+        </geometry>
+    </collision>
+    <xacro:inertial_cylinder mass="0.1" length="0.01" radius="0.01">
+        <origin xyz="0.0 0.0 0.0" rpy="0.0 0.0 0.0"/>
+    </xacro:inertial_cylinder>
+    </link>
+    <gazebo reference="imu_link">
+        <material>Gazebo/White</material>
     </gazebo>
     <!-- CASTER HOLDER JOINT -->
