Commit message: update rover.xacro file

File: bumperbot_ws/src/bumperbot_bringup/urdf/rover.xacro (robot description, xacro)
@@ -66,5 +66,5 @@
         <visual>
             <geometry>
-                <cylinder radius="0.03405" length="0.027"/>
+                <cylinder radius="0.033" length="0.027"/>
                 <!-- <cylinder radius="0.03405" length="0.01"/> -->
             </geometry>
@@ -73,9 +73,9 @@
         <collision>
             <geometry>
-                <cylinder radius="0.03405" length="0.027"/>
+                <cylinder radius="0.033" length="0.027"/>
                 <!-- <sphere radius="0.0325"/> -->
             </geometry>
         </collision>
-        <xacro:inertial_cylinder mass="0.05" length="0.027" radius="0.03405">
+        <xacro:inertial_cylinder mass="0.05" length="0.027" radius="0.033">
             <origin xyz="0.0 0.0 0.0" rpy="0.0 0.0 0.0"/>
         </xacro:inertial_cylinder>
@@ -95,5 +95,5 @@
     <visual>
         <geometry>
-            <cylinder radius="0.03405" length="0.027"/>
+            <cylinder radius="0.033" length="0.027"/>
             <!-- <cylinder radius="0.03405" length="0.01"/> -->
         </geometry>
@@ -102,9 +102,9 @@
     <collision>
         <geometry>
-            <cylinder radius="0.03405" length="0.027"/>
+            <cylinder radius="0.033" length="0.027"/>
             <!-- <sphere radius="0.0325"/> -->
         </geometry>
     </collision>
-    <xacro:inertial_cylinder mass="0.05" length="0.027" radius="0.03405">
+    <xacro:inertial_cylinder mass="0.05" length="0.027" radius="0.033">
         <origin xyz="0.0 0.0 0.0" rpy="0.0 0.0 0.0"/>
     </xacro:inertial_cylinder>
